File: doc/eagle/remote/remote.brd (EAGLE design)
At the start: 25.1 x 48.2 mm, 10 parts

Commit message: Storing metronome params in EEPROM after user inactivity, Eagle files + PDF exports
Connections:
- removed net MT+: C1.1, D1.C, MT24.1
- net 3.3V: now also C1.1, D1.C, MT24.1
Routing:
- net 3.3V: track 46.5 -> 86.3 mm
- net MT+: track 36.7 -> 0.00 mm
Other:
- board text added: "REV2"
- board text removed: "REV1"
Changed lines of the file:
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@@
 <?xml version="1.0" encoding="utf-8"?>
 <!DOCTYPE eagle SYSTEM "eagle.dtd">
-<eagle version="7.7.0">
+<eagle version="9.2.2">
 <drawing>
 <settings>
 <setting alwaysvectorfont="no"/>
+<setting keepoldvectorfont="yes"/>
 <setting verticaltext="up"/>
 </settings>
@@
 <text x="28.0924" y="50.8" size="0.8128" layer="25" font="vector" ratio="20" rot="R90" align="top-center">~D9</text>
 <text x="28.0924" y="40.64" size="0.8128" layer="25" font="vector" ratio="20" rot="R90" align="top-center">3.3V</text>
-<text x="17.78" y="30.48" size="0.8128" layer="25" font="vector" ratio="10">REV1</text>
+<text x="17.78" y="30.48" size="0.8128" layer="25" font="vector" ratio="10">REV2</text>
 </plain>
 <attributes>
@@
 <wire x1="19.05" y1="67.31" x2="20.32" y2="66.04" width="0.4064" layer="16"/>
 <wire x1="20.32" y1="66.04" x2="20.32" y2="59.69" width="0.4064" layer="16"/>
+<contactref element="MT24" pad="1"/>
+<contactref element="D1" pad="C"/>
+<contactref element="C1" pad="1"/>
+<wire x1="26.67" y1="36.83" x2="21.59" y2="36.83" width="0.4064" layer="16"/>
+<wire x1="21.59" y1="36.83" x2="21.59" y2="38.1" width="0.4064" layer="16"/>
+<wire x1="21.59" y1="38.1" x2="17.78" y2="41.91" width="0.4064" layer="16"/>
+<wire x1="17.78" y1="48.26" x2="20.32" y2="50.8" width="0.4064" layer="16"/>
+<wire x1="20.32" y1="50.8" x2="20.32" y2="55.88" width="0.4064" layer="16"/>
+<wire x1="20.32" y1="55.88" x2="22.86" y2="58.42" width="0.4064" layer="16"/>
+<wire x1="22.86" y1="58.42" x2="22.86" y2="64.77" width="0.4064" layer="16"/>
+<wire x1="17.78" y1="41.91" x2="17.78" y2="48.26" width="0.4064" layer="16"/>
+<wire x1="22.86" y1="64.77" x2="21.59" y2="64.77" width="0.4064" layer="16"/>
+<wire x1="21.59" y1="64.77" x2="20.32" y2="66.04" width="0.4064" layer="16"/>
 </signal>
 <signal name="PWM">
@@
 <wire x1="19.05" y1="71.12" x2="16.51" y2="68.58" width="0.4064" layer="16"/>
 </signal>
-<signal name="MT+">
-<contactref element="MT24" pad="1"/>
-<contactref element="D1" pad="C"/>
-<contactref element="C1" pad="1"/>
-<wire x1="26.67" y1="36.83" x2="21.59" y2="36.83" width="0.4064" layer="16"/>
-<wire x1="21.59" y1="36.83" x2="21.59" y2="38.1" width="0.4064" layer="16"/>
-<wire x1="21.59" y1="38.1" x2="17.78" y2="41.91" width="0.4064" layer="16"/>
-<wire x1="17.78" y1="48.26" x2="20.32" y2="50.8" width="0.4064" layer="16"/>
-<wire x1="20.32" y1="50.8" x2="20.32" y2="55.88" width="0.4064" layer="16"/>
-<wire x1="20.32" y1="55.88" x2="22.86" y2="58.42" width="0.4064" layer="16"/>
-<wire x1="22.86" y1="58.42" x2="22.86" y2="64.77" width="0.4064" layer="16"/>
-<wire x1="17.78" y1="41.91" x2="17.78" y2="48.26" width="0.4064" layer="16"/>
-</signal>
 </signals>
