File: doc/eagle/remote/remote.sch (EAGLE design)
At the start: 10 parts

Commit message: Storing metronome params in EEPROM after user inactivity, Eagle files + PDF exports
Connections:
- removed net MT+: C1.1, D1.C, MT24.1
- net 3.3V: now also C1.1, D1.C, MT24.1
Changed lines of the file:
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@@
 <?xml version="1.0" encoding="utf-8"?>
 <!DOCTYPE eagle SYSTEM "eagle.dtd">
-<eagle version="7.7.0">
+<eagle version="9.2.2">
 <drawing>
 <settings>
 <setting alwaysvectorfont="no"/>
+<setting keepoldvectorfont="yes"/>
 <setting verticaltext="up"/>
 </settings>
@@
 <schematic xreflabel="%F%N/%S.%C%R" xrefpart="/%S.%C%R">
 <attributes>
+<attribute name="CNAME" value="Metronom - remote module"/>
+<attribute name="CREVISION" value="2"/>
+<attribute name="DESIGNER" value="Piotr Wysocki"/>
 </attributes>
 <variantdefs>
@@
 <part name="R3" library="rcl" deviceset="R-EU_" device="0204/7" value="10k"/>
 <part name="Q2" library="transistors" deviceset="2N700*" device="_TO92" technology="0"/>
+<part name="FRAME1" library="SparkFun-Aesthetics" library_urn="urn:adsk.eagle:library:507" deviceset="FRAME-A4L" device=""/>
 </parts>
 <sheets>
@@
 <attribute name="VALUE" x="80.264" y="64.516" size="1.778" layer="96"/>
 </instance>
+<instance part="FRAME1" gate="G$1" x="-93.98" y="-15.24" smashed="yes">
+<attribute name="SHEET" x="101.6" y="-13.97" size="2.54" layer="94" font="vector"/>
+<attribute name="CNAME" x="87.63" y="1.27" size="2.54" layer="94" font="vector"/>
+<attribute name="CREVISION" x="140.94" y="-14.07" size="2.54" layer="94" font="vector"/>
+<attribute name="DESIGNER" x="132.28" y="-8.89" size="2.54" layer="94" font="vector"/>
+</instance>
 </instances>
 <busses>
@@
 <wire x1="-7.62" y1="71.12" x2="2.54" y2="71.12" width="0.1524" layer="91"/>
 <label x="-7.62" y="71.12" size="1.778" layer="95"/>
+</segment>
+<segment>
+<pinref part="MT24" gate="G$1" pin="1"/>
+<wire x1="83.82" y1="83.82" x2="83.82" y2="96.52" width="0.1524" layer="91"/>
+<wire x1="83.82" y1="96.52" x2="73.66" y2="96.52" width="0.1524" layer="91"/>
+<pinref part="D1" gate="1" pin="C"/>
+<wire x1="73.66" y1="96.52" x2="63.5" y2="96.52" width="0.1524" layer="91"/>
+<wire x1="63.5" y1="96.52" x2="63.5" y2="91.44" width="0.1524" layer="91"/>
+<pinref part="C1" gate="G$1" pin="1"/>
+<wire x1="73.66" y1="93.98" x2="73.66" y2="96.52" width="0.1524" layer="91"/>
+<junction x="73.66" y="96.52"/>
+<label x="86.36" y="88.9" size="1.778" layer="95"/>
+<pinref part="SUPPLY3" gate="G$1" pin="3.3V"/>
+<wire x1="73.66" y1="101.6" x2="73.66" y2="96.52" width="0.1524" layer="91"/>
 </segment>
 </net>
@@
 </segment>
 </net>
-<net name="MT+" class="0">
-<segment>
-<pinref part="MT24" gate="G$1" pin="1"/>
-<wire x1="83.82" y1="83.82" x2="83.82" y2="96.52" width="0.1524" layer="91"/>
-<wire x1="83.82" y1="96.52" x2="73.66" y2="96.52" width="0.1524" layer="91"/>
-<pinref part="D1" gate="1" pin="C"/>
-<wire x1="73.66" y1="96.52" x2="63.5" y2="96.52" width="0.1524" layer="91"/>
-<wire x1="63.5" y1="96.52" x2="63.5" y2="91.44" width="0.1524" layer="91"/>
-<pinref part="C1" gate="G$1" pin="1"/>
-<wire x1="73.66" y1="93.98" x2="73.66" y2="96.52" width="0.1524" layer="91"/>
-<junction x="73.66" y="96.52"/>
-<pinref part="SUPPLY3" gate="G$1" pin="3.3V"/>
-<wire x1="73.66" y1="101.6" x2="73.66" y2="96.52" width="0.1524" layer="91"/>
-<label x="86.36" y="88.9" size="1.778" layer="95"/>
-</segment>
-</net>
 </nets>
 </sheet>
@@
 </schematic>
 </drawing>
+<compatibility>
+<note version="8.2" severity="warning">
+Since Version 8.2, EAGLE supports online libraries. The ids
+of those online libraries will not be understood (or retained)
+with this version.
+</note>
+<note version="8.3" severity="warning">
+Since Version 8.3, EAGLE supports URNs for individual library
+assets (packages, symbols, and devices). The URNs of those assets
+will not be understood (or retained) with this version.
+</note>
+</compatibility>
 </eagle>
